File: FCU-V10A/Connector.kicad_sch (KiCad schematic)
At the start: 0 parts

Commit message: Connector
Parts:
- added J2, J3, J4, J5: Conn_01x03_Pin, Connector_PinHeader_2.54mm:PinHeader_1x03_P2.54mm_Horizontal, symbol Connector:Conn_01x03_Pin
Connections:
- new net +3.3V: J2.1 (Pin_1), J3.1 (Pin_1), J4.1 (Pin_1), J5.1 (Pin_1)
- new net GND: J2.3 (Pin_3), J3.3 (Pin_3), J4.3 (Pin_3), J5.3 (Pin_3)
Other:
- note added: "ESC"
